File: HomeyPCB/HomeyPCB.kicad_pcb (KiCad board)
At the start: 2 copper layers, 99 x 90 mm, 99 parts, among them J1 Barrel_Jack, J6 USB_C_Receptacle_USB2.0_14P, J7 SERVO1/2, Q1 AO3400A_C42419946, Q2 AO3400A_C42419946, Q3 AO3400A_C42419946, Q4 AO3400A_C42419946, SW1 BOOT, SW2 RESET, U1 ESP32-WROOM-32E, U10 I2, U11 PC817C_C20612449, U12 I3, U13 PC817C_C20612449, U14 I4, U15 PC817C_C20612449, U16 CH340C, U17 LM66100DCKR, U18 189RV0036, U19 SUPPLY, U2 LAN8720A-CP-TR, U20 AMS1117-3.3_C6067465, U21 LM66100DCKR, U22 LM2596S-5.0_C5276750, U23 LM66100DCKR, U3 DP1435-5V, U4 1O, U5 2O, U6 3O, U7 4O, U8 PC817C_C20612449, U9 I1, X1 X322525MOB4SI

Commit message: ee2
Parts:
- moved L1 0.31 mm to (214.3, 81.9)
Connections:
- BUZZER1 pad 1: GPIO34 -> GPIO32
- D7 pad 2: GPIO36 -> GPIO4
- R11 pad 1: GPIO35 -> GPIO14
- U1 pad 31: TXEN -> TXDO
- U1 pad 36: GPIO22 -> TXD1
- U1 pad 37: GPIO23 -> MDC
- U13 pad 3: GPIO23 -> GPIO34
- U15 pad 3: GPIO14 -> GPIO35
- U8 pad 3: GPIO22 -> GPIO37
Routing:
- net TXDO: track 0.00 -> 209.4 mm, vias 0 -> 8
- net TXD1: track 0.00 -> 170.0 mm, vias 0 -> 9
- net GPIO36: track 139.1 -> 0.00 mm, vias 2 -> 0
- net MDC: track 0.00 -> 133.2 mm, vias 0 -> 4
- net GPIO4: track 0.00 -> 103.7 mm, vias 0 -> 4
- net GPIO37: track 0.00 -> 64.3 mm, vias 0 -> 4
- net GPIO22: track 55.9 -> 0.00 mm, vias 1 -> 0
- net TXEN: track 107.3 -> 162.5 mm, vias 2 -> 4
- net GPIO23: track 46.3 -> 0.00 mm, vias 2 -> 0
- net GPIO32: track 0.00 -> 45.4 mm, vias 0 -> 1
- net GPIO35: track 19.4 -> 48.1 mm
- net GPIO14: track 39.7 -> 11.8 mm, vias 2 -> 3
- net GPIO34: track 47.7 -> 58.7 mm, vias 1 -> 7
- net RXD1/MODE1: track 62.9 -> 66.4 mm
- net ETH_CLK: track 107.9 -> 111.0 mm
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