File: HomeyPCB/HomeyPCB.kicad_sch (KiCad schematic)
At the start: 95 parts, among them J1 Barrel_Jack, J6 USB_C_Receptacle_USB2.0_14P, J7 SERVO1/2, Q1 AO3400A_C42419946, Q2 AO3400A_C42419946, Q3 AO3400A_C42419946, Q4 AO3400A_C42419946, SW1 BOOT, SW2 RESET, U1 ESP32-WROOM-32E, U10 I2, U11 PC817C_C20612449, U12 I3, U13 PC817C_C20612449, U14 I4, U15 PC817C_C20612449, U16 CH340C, U17 LM66100DCKR, U18 189RV0036, U19 SUPPLY, U2 LAN8720A-CP-TR, U20 AMS1117-3.3_C6067465, U21 LM66100DCKR, U22 LM2596S-5.0_C5276750, U23 LM66100DCKR, U3 DP1435-5V, U4 1O, U5 2O, U6 3O, U7 4O, U8 PC817C_C20612449, U9 I1, X1 X322525MOB4SI

Commit message: ee2
Connections:
- net GPIO14: now also R11.1; no longer U15.3 (EM)
- net GPIO32: now also BUZZER1.1
- net GPIO34: now also U13.3 (EM); no longer BUZZER1.1
- net GPIO35: now also U15.3 (EM); no longer R11.1
- net GPIO36: no longer D7.2 (DIN)
- net GPIO37: now also U8.3 (EM)
- net GPIO4: now also D7.2 (DIN)
- net MDC: now also U1.37 (IO23)
- net TXD1: now also U1.36 (IO22)
- net TXDO: now also U1.31 (IO19)
- net TXEN: no longer U1.31 (IO19)
- removed net GPIO22: U1.36 (IO22), U8.3 (EM)
- removed net GPIO23: U1.37 (IO23), U13.3 (EM)
